Commit message: PR06 defect: attach lidar to camera frame

File: src/course_description/urdf/vehicle.urdf.xacro (robot description, xacro)
@@ -80,5 +80,5 @@
   </link>
   <joint name="lidar_joint" type="fixed">
-    <parent link="base_link"/><child link="lidar_link"/>
+    <parent link="camera_link"/><child link="lidar_link"/>
     <origin xyz="${sensor_x} 0 ${sensor_z}" rpy="0 0 0"/>
   </joint>
